File: rc2014_nvram.kicad_pcb (KiCad board)
At the start: 2 copper layers, 99.1 x 49.9 mm, 13 parts, among them U1 CY62256-70PC, U2 74LS32, U3 CY62256-70PC, U6 74HCT04

Commit message: Fix grounding issues
Parts:
- R1: value R -> 10K
- U3: renamed from BQ2201SN-N1; value ~ -> BQ2201SN
- U4: renamed from BQ2201SN-N2; value ~ -> BQ2201SN
- U5: renamed from U2; value 74LS32 -> 74HTC32
- moved C1 28.1 mm to (135.5, 112.2), turned to 0 degrees
- moved U4 22.6 mm to (137.0, 107.5)
- moved C3 22.5 mm to (131.0, 84.0)
- moved U3 22.5 mm to (137.0, 85.2)
- moved U1 21.5 mm to (145.0, 101.5)
- moved U2 15.8 mm to (145.0, 119.2)
- renumbered U3 to U2
Connections:
- U1 pad 11: /D0 -> /D2
- U1 pad 12: /D1 -> /D4
- U1 pad 13: /D2 -> /D6
- U1 pad 15: /D3 -> /D7
- U1 pad 16: /D4 -> /D5
- U1 pad 17: /D5 -> /D3
- U1 pad 18: /D6 -> /D1
- U1 pad 19: /D7 -> /D0
- U1 pad 2: /A12 -> /A13
- U1 pad 21: /A10 -> /A3
- U1 pad 23: /A11 -> /A6
- U1 pad 24: /A9 -> /A8
- U1 pad 25: /A8 -> /A10
- U1 pad 26: /A13 -> /A12
- U1 pad 3: /A7 -> /A11
- U1 pad 4: /A6 -> /A9
- U1 pad 5: /A5 -> /A7
- U1 pad 6: /A4 -> /A5
- U1 pad 7: /A3 -> /A4
- U2 pad 11: /D0 -> /D2
- U2 pad 12: /D1 -> /D4
- U2 pad 13: /D2 -> /D6
- U2 pad 15: /D3 -> /D7
- U2 pad 16: /D4 -> /D5
- U2 pad 17: /D5 -> /D3
- U2 pad 18: /D6 -> /D1
- U2 pad 19: /D7 -> /D0
- U2 pad 2: /A12 -> /A13
- U2 pad 21: /A10 -> /A3
- U2 pad 23: /A11 -> /A6
- U2 pad 24: /A9 -> /A8
- U2 pad 25: /A8 -> /A10
- U2 pad 26: /A13 -> /A12
- U2 pad 3: /A7 -> /A11
- U2 pad 4: /A6 -> /A9
- U2 pad 5: /A5 -> /A7
- U2 pad 6: /A4 -> /A5
- U2 pad 7: /A3 -> /A4
Routing:
- net GND: track 289.5 -> 476.4 mm, vias 3 -> 20
- net /A15: track 81.8 -> 57.7 mm, vias 1 -> 0
- net Net-(U4-~{CE}): track 34.5 -> 10.9 mm, vias 0 -> 1
- net /A11: track 103.7 -> 81.5 mm, vias 2 -> 0
- net /A6: track 70.5 -> 92.1 mm
- net /A3: track 70.5 -> 89.9 mm
- net /A12: track 80.7 -> 98.1 mm
- net /A9: track 96.4 -> 79.4 mm, vias 2 -> 0
- net /D4: track 56.2 -> 40.0 mm, vias 1 -> 0
- net /A13: track 97.9 -> 83.6 mm, vias 1 -> 0
- net /D0: track 45.1 -> 59.4 mm
- net Net-(U5-Pad10): track 41.2 -> 27.5 mm, vias 1 -> 0
- net /D1: track 46.1 -> 59.2 mm
- net /D6: track 48.2 -> 37.0 mm, vias 1 -> 0
- net /A1: track 70.5 -> 81.4 mm, vias 0 -> 3
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Other:
- board text added: "1"
- board text added: "NVRAM V 1.1 github.com/jce/rc2014_nvram"

Commit message: V 1.1, second proto run
Routing:
- net GND: track 476.4 -> 863.2 mm, vias 20 -> 44
- net Net-(U2-VCC): track 9.87 -> 8.25 mm
- net Net-(U2-~{CS}): track 42.2 -> 42.7 mm
Other:
- board text added: "NVRAM V 1.1 github.com/jce/nvram_for_rc2014"
- board text removed: "NVRAM V 1.1 github.com/jce/rc2014_nvram"
